File: pds019_main_082_ext.sch (EAGLE design)
At the start: 400 parts, among them CN1 2EDGRM-7.62-03P, CN10 ST-033, CN11 KF2-EDGRHM-3.81-02P, CN12 BH-10, CN13 BH14, CN2 B5P-VH, CN3 B5P-VH, CN4 KF2EDGRHM-5.08-2X2P, CN5 KF2EDGRHM-5.08-2x3P, CN6 KF2EDGRHM-5.08-2x3P, CN7 COAX_FBNC_JR_CHN, CN8 COAX_FBNC_JR_CHN, CN9 USBA-KLS1-191-4P-0.7, J4.1 CONN_PAD-1,5R, J4.2 CONN_PAD-1,5R, J5.1 CONN_PAD-1,5R, J5.2 CONN_PAD-1,5R, K1 HLS8-22F-DC12V-C, K2 HLS8-22F-DC12V-C, K3 HLS8-22F-DC12V-C, K4 HLS8-22F-DC12V-C, K5 HLS8-22F-DC12V-C, K6 SLC-12VDC-SL-C, M1 MPAD3,2-8, M10 MPAD3,2-5,5, M11 MPAD3,2-5,5, M12 MPAD3,2-5,5, M13 MPAD3,2-5,5, M14 MPAD3,2-5,5, M17 MPAD3,2-5,5, M18 MPAD3,2-5,5, M19 MPAD3,2-5,5, M2 MPAD3,2-8, M20 MPAD3,2-5,5, M21 MPAD3,2-5,5, M3 MPAD3,2-8, M4 MPAD3,2-8, M5 MPAD3,2-8, M7 MPAD3,2-8, M8 MPAD3,2-8, M9 MPAD3,2-8, Q1 NC, Q2 BCR133, Q3 NC, Q4 NC, U1 STM32F2xxR, U10 74LVC1G07, U11 TL431, U12 TL431, U13 AD8667R, U14 AD8667R, U15 REF3020AIDBZ, U16 REF3020AIDBZ, U17 MCP3551SN, U18 MCP3551SN, U19 P2AU-0505ELF, U2 ESP32-WROVER-E, U20 P2AU-0505ELF, U21 ISO7231CDW, U22 ISO7231CDW, U23 NC, U24 NC, U25 NC, U26 74AHCT1G125DBV, U27 3.3V, U28 K78-1000R, U29 K78-1000R, U3 ULN2003AD, U30 74LVC1G17, U31 TPS2553DBV, U4 TPS54231DDR, U5 TPS563201DDC, U6 B1224LS-1WR3, U7 LM293D, U8 74LVC1G14DBV, U9 MAX809S, X1 PLS-04, X11 WF-3, X3 PLS-05, X4 PLD-06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

Commit message: some progress
Parts:
- removed CN3: B5P-VH, pds019_main_082_ext:CONN_LNPE-JST-B5P-VH
- removed CN5, CN6: KF2EDGRHM-5.08-2x3P, pds019_main_082_ext:TBLOCK_2X03P-KF2-EDGRHM-5.08-2X3P
- removed HL17: LED-0805, pds019_main_082_ext:LED-0805
- removed PC1: KPC357NT0C, pds019:PC817E-MINIFLAT4
- removed U4: TPS54231DDR, pds019_main_082_ext:TPS54231DDR
- removed X4: PLD-06, pds019_main_082_ext:PLD-06
- removed X6: (no value), pds019_main_082_ext:JP1E
- added CON1: PINHEAD_2X03-PTH-2.54, pinhead:PINHEAD_2X03-PTH-2.54
- added CON2: CON-5P-JST-VH, Connectors:CON-5P-JST-VH
- added CON3, CON4: CON-2X3, degson:CON-2X3
- added IC1: TPS54231, dc-dc:TPS54231
- added IC2: KPC357NT-SOP-4, misc:KPC357NT-SOP-4
- added LED1: LED-0805, rc:LED-0805
- added X10: PINHEAD_1X02-2.54, pinhead:PINHEAD_1X02-2.54
- BAT1: value CR2032 -> BATTERY-L-KLS5-CR2032-01; device pds019_main_082_ext:CR2032-H -> mechanical:BATTERY-L-KLS5-CR2032-01
- C33, C34: device pds018:C1812 -> rc:C-1812; PKG 1812 -> (none)
- C89: device pds018:C0603 -> rc:C-0603; PKG 0603 -> (none); TOL -20/+80% -> (none); TYPE Y5V -> (none)
- CN1: device pds019_main_082_ext:TBLOCK_03P-KF2EDGRM-7.62 -> degson:CON-3P-2EDGRM-7.62
- CN10: device pds019:ST-033_DCI -> Connectors:ST-033
- CN2: value B5P-VH -> CON-5P-JST-VH; device pds019_main_082_ext:CONN_SW_LN-B5P-VH(-1) -> Connectors:CON-5P-JST-VH
- CN4: value KF2EDGRHM-5.08-2X2P -> CON-2X2; device pds019_main_082_ext:TBLOCK_2X02P-KF2-EDGRHM-5.08-2X2P -> degson:CON-2X2
- CN7, CN8: value COAX_FBNC_JR_CHN -> RF_CONNECTOR-BNC-KY-WE; device pds019:COAX_FBNC_JR_CHN -> Connectors:RF_CONNECTOR-BNC-KY-WE
- D1, D5: device pds019:SMAJ5.0A -> TVS_diodes:SMAJ5.0A
- D6: device pds019_main_082_ext:SS14-SMA -> Diodes:SS34
- D8: device pds019_main_082_ext:SMBJ -> TVS_diodes:SMBJ15A-SMB
- F1, F2, F3, F4, F5, F6, F7, F8, F9: device pds019_main_082_ext:FUSE_HOLDER_FC-001S -> rc:FUSE-FC-001S
- F10: value 500mA -> FUSE-1206; device pds019_main_082_ext:FUSE-SMD-1206 -> rc:FUSE-1206; CURRENT (none) -> 500 mA
- F11: device pds019:FUSE-SMD-1206 -> rc:FUSE-1206
- K1, K2, K3, K4, K5: device pds019_main_082_ext:SRD-U -> misc:SRD-U
- Q4: device pds019:IRLML2244 -> mosfet:IRLML2244
- U10: value 74LVC1G07 -> 74LVC1G07GV; device pds019:74LVC1G07 -> misc:74LVC1G07GV
- U11, U12: device pds019:TL431-SOT-23 -> misc:TL431
- U13, U14: value AD8667R -> AD8667ARZ-SO8; device pds019:AD8667R -> misc:AD8667ARZ-SO8
- U15: device pds019:REF3020AIDBZ -> misc:REF3020AIDBZ
- U16: device pds019:REF3020AIDBZ -> misc:REF3020AIDBZ; MF TI -> (none); PKG SOT-23 -> (none); VOLT 2.048V -> (none)
- U17, U18: value MCP3551SN -> MCP3550; device pds019:MCP3551SN -> misc:MCP3550
- U19, U20: value P2AU-0505ELF -> B0503S-1WR3; device pds018:P2AU-0505ELF -> dc-dc:B0503S-1WR3
- U2: value ESP32-WROVER-E -> ESP32-WROVER-(I)E; device pds019_main_082_ext:ESP32-WROVER-(I)E -> ali_modules:ESP32-WROVER-(I)E
- U21, U22: device pds018:ADUM1301 -> serial_interfaces:ADUM1301
- U25: device pds019_main_082_ext:74LVC1T45DBV -> misc:SN74LVC1T45DBV
- U26: value 74AHCT1G125DBV -> SN74AHCT1G125DBVR-SOT23-5; device pds019_main_082_ext:74AHCT1G125DBV -> misc:SN74AHCT1G125DBVR-SOT23-5
- U30: device pds019:74LVC1G07 -> misc:74LVC1G17; PKG SOT23-5 -> (none)
- U31: device pds019:TPS2553DBV -> misc:TPS2553DBV
- U7: device pds019:LM393D -> misc:LM293D-SO8
- U8: device pds019:74LVC1G08DBV -> misc:74LVC1G14DBV
- U9: device pds019_main_082_ext:MAX809S -> misc:MAX809S
- X1: value PLS-04 -> PINHEAD_1X04-2.54; device pds018:PLS-04 -> pinhead:PINHEAD_1X04-2.54
- X2, X9: value (none) -> PINHEAD_1X02-2.54; device pds019_main_082_ext:JP1E -> pinhead:PINHEAD_1X02-2.54
- X3: value PLS-05 -> PINHEAD_1X05-2.54; device pds019_main_082_ext:PLS-05 -> pinhead:PINHEAD_1X05-2.54
- X5: value PLS-03 -> PINHEAD_1X03-2.54; device pds019:PLS-03 -> pinhead:PINHEAD_1X03-2.54
- X7, X8: value PLS-03 -> PINHEAD_1X03-2.54; device pds019_main_082_ext:PLS-03 -> pinhead:PINHEAD_1X03-2.54
Connections:
- net +12V: now also IC1.VIN; no longer U4.VIN
- net +3V3: now also CON1.1, IC2.COLLECTOR, X1.4; no longer PC1B.C, X1.1, X4.1
- net AC_N: now also CN2.5, CON3.1.2, CON3.2.2, CON4.1.2, CON4.2.2; no longer CN2.NI, CN5.1.2, CN5.2.2, CN6.1.2, CN6.2.2
- net ENC_BTN: now also X10.1; no longer X6.1
- net ESP32_STM_SWCLK: now also U2.IO22; no longer U2.IO22/VSPIWP/RTS0
- net ESP32_STM_SWDIO: now also U2.IO21; no longer U2.IO21/VSPIHD
- net GND: now also BAT1.NEGATIVE, CON1.6, IC1.GND, LED1.C, U10.GND, U19.IN-, U2.GND, U20.IN-, U30.GND, U8.GND, X1.1, X10.2; no longer BAT1.-, HL17.K, U10.VSS, U19.VIN-, U2.GND@1, U2.GND@15, U2.GND@38, U2.GND@39, U20.VIN-, U30.VSS, U4.EP, U4.GND, U8.VSS, X1.4, X4.6, X6.2
- net LVL_24V: now also IC2.A; no longer PC1A.A
- net LVL_GND: now also U7B.IN+, U7B.IN-; no longer U7B.+IN, U7B.-IN
- net MTCK: now also U2.IO13; no longer U2.IO13/MTCK/HSPID
- net MTDI: now also U2.IO12; no longer U2.IO12/MTDI/HSPIQ
- net MTDO: now also U2.IO15; no longer U2.IO15/MTDO/HSPICS0
- net MTMS: now also U2.IO14; no longer U2.IO14/MTMS/HSPICLK
- net N$10: now also LED1.A; no longer HL17.A
- net N$12: now also CN7.ANT; no longer CN7.CEN
- net N$124: now also CON1.5; no longer X4.5
- net N$13: now also CN8.ANT; no longer CN8.CEN
- net N$149: now also IC1.BOOT; no longer U4.BOOT
- net N$150: now also CON1.2; no longer X4.2
- net N$165: now also F11.2; no longer F11.P$2
- net N$19: now also X1.3; no longer X1.2
- net N$190: now also IC1.PH; no longer U4.PH
- net N$192: now also IC1.COMP; no longer U4.COMP
- net N$20: now also X1.2; no longer X1.3
- net N$204: now also CON4.1.1; no longer CN5.1.1
- net N$205: now also IC1.VSENSE; no longer U4.VSENSE
- net N$207: now also IC1.EN; no longer U4.EN
- net N$211: now also CON4.2.1; no longer CN5.2.1
- net N$213: now also CON1.3; no longer X4.3
- net N$214: now also CON3.1.1; no longer CN6.1.1
- net N$216: now also CON1.4; no longer X4.4
- net N$217: now also CON3.2.1; no longer CN6.2.1
- net N$23: now also IC2.C; no longer PC1A.C
- net N$29: now also F11.1; no longer F11.P$1
- net N$34: now also U19.OUT+; no longer U19.VOUT+
- net N$35: now also U2.IO36; no longer U2.IO36/SENS_VP
- net N$36: now also U2.IO39; no longer U2.IO39/SENS_VN
- net N$40: now also U7A.IN-; no longer U7A.-IN
- net N$42: now also U19.OUT-; no longer U19.VOUT-
- net N$46: now also U2.IO19; no longer U2.IO19/VSPIQ
- net N$47: now also U2.IO18; no longer U2.IO18/VSPICLK
- net N$48: now also U2.IO5; no longer U2.IO5/VSPICS0
- net N$49: no longer U2.NC@28
- net N$50: no longer U2.NC@27
- net N$51: now also U2.IO4; no longer U2.IO4/HSPID
- net N$52: now also U2.IO2; no longer U2.IO2/HSPIWP
- net N$53: now also U20.OUT+; no longer U20.VOUT+
- net N$55: now also U20.OUT-; no longer U20.VOUT-
- net N$6: now also CN2.1; no longer CN2.LI
- net N$64: now also F10.1; no longer F10.P$1
- net N$68: now also U19.IN+; no longer U19.VIN+
- net N$69: now also IC1.SS; no longer U4.SS
- net N$7: now also CN2.2, CON2.3; no longer CN2.LO, CN3.L
- net N$70: now also U20.IN+; no longer U20.VIN+
- net N$73: now also U7A.IN+; no longer U7A.+IN
- net N$8: now also CN2.4, CON2.1; no longer CN2.NO, CN3.N
- net N$89: no longer U8.B
- net N$9: now also U2.IO23; no longer U2.IO23/VSPID
- net N$96: now also F10.2; no longer F10.P$2
- net PE: now also CON2.5, CON3.1.3, CON3.2.3, CON4.1.3, CON4.2.3; no longer CN3.PE, CN5.1.3, CN5.2.3, CN6.1.3, CN6.2.3
- net PH_VCOM: now also CN7.GND; no longer CN7.SH
- net RTC_VBAT: now also BAT1.POSITIVE; no longer BAT1.+
- net RX_COM: now also CN8.GND; no longer CN8.SH
- net SENSOR_LEVEL: now also IC2.EMITTER; no longer PC1B.E
Other:
- note added: "У CN2/CN3 были странные футпринты с недостающими пинами. Я заменил на обычные"
- note removed: "Vfb=0.8V"

Commit message: its done now
Parts:
- removed CN9: USBA-KLS1-191-4P-0.7, pds019_main_082_ext:USBA-KLS1-191-4P-0.7
- removed K6: SLC-12VDC-SL-C, pds019_main_082_ext:SLC-12VDC-SL-C
- removed LCD1: LCD12864, pds019_main_082_ext:LCD12864
- added CON5: USB-A-KLS1-191, Connectors:USB-A-KLS1-191
- added CON6: PINHEAD_1X20-2.54-MALE-LONG, pinhead:PINHEAD_1X20-2.54-MALE-LONG
- added K7: SRD-SLC, misc:SRD-SLC
- C108: value 4700pF 2kV -> 4700pF; device pds019_main_082_ext:C-5MM -> rc:C-RADIAL-5MM; VOLTAGE (none) -> 2kV
- C35, C36: value 1000pF 2kV -> 1000pF; device pds019:C-5MM -> rc:C-RADIAL-5MM; VOLTAGE (none) -> 2kV
- C59: value 100,0 25V -> 100,0; device pds019_main_082_ext:CTANT7X4 -> rc:CPOL-SMD-TYPE-D; PACKAGE (none) -> TYPE D; PKG SMD D -> (none); TOL 20% -> (none); TYPE TANT -> (none); VOLT 10V -> (none); VOLTAGE (none) -> 25V
- C60: value 100,0 6V3 -> 100,0; device pds019_main_082_ext:CTANT_B -> rc:CPOL-TANT-TYPE-B; PACKAGE (none) -> TYPE B; VOLTAGE (none) -> 6.3V
- C72: value 150,0 16V -> 150,0; device pds019_main_082_ext:CTANT7X4 -> rc:CPOL-SMD-TYPE-D; PACKAGE (none) -> TYPE D; PKG SMD D -> (none); TOL 20% -> (none); TYPE TANT -> (none); VOLT 10V -> (none); VOLTAGE (none) -> 16V
- C90: value 4700pF 2kV -> 4700pF; device pds019:C-5MM -> rc:C-RADIAL-5MM; VOLTAGE (none) -> 2kV
- CN12: device pds019_main_082_ext:IDC_CONN10-BH10 -> Connectors:IDC_CONN10-BH10
- CN13: device pds019_main_082_ext:IDC_CONN14-BH14 -> Connectors:IDC_CONN14-BH14
- ENC1: device pds019_main_082_ext:ENC-PEC12R-4XXXF-SXXXX -> misc:ENC-PEC12R-4XXXF-SXXXX
- L1: value 22uH 0630 -> 22uH; device pds019_main_082_ext:L-SMD06030 -> power_inductors:22µH-0630
- L2: value 2,2uH 0520 -> 3.3uH; device pds019_main_082_ext:L-SMD05020 -> power_inductors:3.3µH-0520
- Q1, Q2, Q3: device pds018:BCR133 -> misc:BCR133; MF NXP -> (none); PKG SOT23-3 -> (none)
- SB1: device pds019_main_082_ext:SW_BUTTON -> mechanical:TACT_SWITCH-6X6-PTH
- U1: device pds019_main_082_ext:STM32F205R-MIL -> stm32:STM32F205RBT6
- U6: device pds019:MOSNSUN_B1224LS-1WR3 -> dc-dc:B1224LS-1WR3
- VR1: device pds019_main_082_ext:S20K420 -> rc:VARISTOR-22MM; MANF (none) -> KLS; MANF# (none) -> L-KLS6-20D431K
- Z1: value 25MHz 3225 -> 25MHz; device pds019_main_082_ext:CRYSTAL-3225_4PIN -> crystal:CRYSTAL-4P-24MHZ-3.2X2.5
- Z2: value 32K 3215 -> 32K; device pds019_main_082_ext:XTAL-3215 -> crystal:CRYSTAL-2P-32X15
Connections:
- net !LCD_RST: now also CON6.17; no longer LCD1.!RST
- net +12V: now also K7C.2, U6.IN+; no longer K6.1.2, U6.VIN+
- net AC_L: now also K7A.COM; no longer K6.2.COM
- net ENC_BTN: now also U1.PC13; no longer U1.PC13_RTC_AF1
- net ESP32_RXD0: now also U1.PA0; no longer U1.PA0_WKUP
- net GND: now also CON5.GND, CON6.1, CON6.15, U6.IN-, Z1.GND; no longer CN9.GND, CN9.S1, CN9.S2, LCD1.PSB/CS1, LCD1.VSS, U6.VIN-, Z1.P$2
- net LCD_CS: now also CON6.4; no longer LCD1.RS/CS
- net LCD_DATA: now also CON6.5; no longer LCD1.RW/SID
- net LCD_LED_A: now also CON6.19; no longer LCD1.A
- net LCD_LED_K: now also CON6.20; no longer LCD1.K
- net LCD_V0: now also CON6.3; no longer LCD1.V0
- net LCD_VEE: now also CON6.18; no longer LCD1.VEE
- net LVL_24V: now also U6.OUT+; no longer U6.VOUT+
- net LVL_GND: now also U6.OUT-; no longer U6.VOUT-
- net N$125: now also CON5.D-; no longer CN9.D-
- net N$131: now also CON5.D+; no longer CN9.D+
- net N$18: now also CON6.6; no longer LCD1.E/CLK
- net N$183: now also K7A.NO; no longer K6.2.NO
- net N$30: now also CON6.2; no longer LCD1.VDD
- net N$39: now also K7C.1; no longer K6.1.1
- net N$63: now also Z1.1; no longer Z1.P$1
- net N$64: now also CON5.VBUS; no longer CN9.VBUS
- net OSC_IN: now also U1.PH0, Z1.2; no longer U1.PH0_OSC_IN, Z1.P$3
- net OSC_OUT: now also U1.PH1; no longer U1.PH1_OSC_OUT
- net RTC_XTAL_IN: now also U1.PC14; no longer U1.PC14_OSC32_IN
- net RTC_XTAL_OUT: now also U1.PC15; no longer U1.PC15_OSC32_OUT
Other:
- note added: "Модель разъема CN11 не найти. Да и вообще документацию про него не найти"
- moved on the sheet: BAT1, BZ1, C1, C10, C107, C109, C11, C110, C111, C12, C13, C14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
