File: pds019_main_082_ext.brd (EAGLE design)
At the start: 255 x 178.4 mm, 408 parts, among them CN1 2EDGRM-7.62-03P, CN10 ST-033, CN11 KF2-EDGRHM-3.81-02P, CN12 BH-10, CN13 BH14, CN2 B5P-VH, CN3 B5P-VH, CN4 KF2EDGRHM-5.08-2X2P, CN5 KF2EDGRHM-5.08-2x3P, CN6 KF2EDGRHM-5.08-2x3P, CN7 COAX_FBNC_JR_CHN, CN8 COAX_FBNC_JR_CHN, CN9 USBA-KLS1-191-4P-0.7, J4.1 CONN_PAD-1,5R, J4.2 CONN_PAD-1,5R, J5.1 CONN_PAD-1,5R, J5.2 CONN_PAD-1,5R, K1 HLS8-22F-DC12V-C, K2 HLS8-22F-DC12V-C, K3 HLS8-22F-DC12V-C, K4 HLS8-22F-DC12V-C, K5 HLS8-22F-DC12V-C, K6 SLC-12VDC-SL-C, M1 MPAD3,2-8, M10 MPAD3,2-5,5, M11 MPAD3,2-5,5, M12 MPAD3,2-5,5, M13 MPAD3,2-5,5, M14 MPAD3,2-5,5, M17 MPAD3,2-5,5, M18 MPAD3,2-5,5, M19 MPAD3,2-5,5, M2 MPAD3,2-8, M20 MPAD3,2-5,5, M21 MPAD3,2-5,5, M3 MPAD3,2-8, M4 MPAD3,2-8, M5 MPAD3,2-8, M7 MPAD3,2-8, M8 MPAD3,2-8, M9 MPAD3,2-8, Q1 NC, Q2 BCR133, Q3 NC, Q4 NC, U1 STM32F2xxR, U10 74LVC1G07, U11 TL431, U12 TL431, U13 AD8667R, U14 AD8667R, U15 REF3020AIDBZ, U16 REF3020AIDBZ, U17 MCP3551SN, U18 MCP3551SN, U19 P2AU-0505ELF, U2 ESP32-WROVER-E, U20 P2AU-0505ELF, U21 ISO7231CDW, U22 ISO7231CDW, U23 NC, U24 NC, U25 NC, U26 74AHCT1G125DBV, U27 3.3V, U28 K78-1000R, U29 K78-1000R, U3 ULN2003AD, U30 74LVC1G17, U31 TPS2553DBV, U4 TPS54231DDR, U5 TPS563201DDC, U6 B1224LS-1WR3, U7 LM293D, U8 74LVC1G14DBV, U9 MAX809S, X1 PLS-04, X11 WF-3, X3 PLS-05, X4 PLD-06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

Commit message: some progress
Parts:
- removed CN3: B5P-VH, pds019_main_082_ext:JST_B5P_VH(-2)
- removed CN5, CN6: KF2EDGRHM-5.08-2x3P, pds019_main_082_ext:KF2EDRHM-5.08-2X3P
- removed HL17: LED-0805, pds019_main_082_ext:LED0805
- removed PC1: KPC357NT0C, pds019:MINIFLAT_4PIN
- removed U4: TPS54231DDR, pds019_main_082_ext:SO08-EP_MAX
- removed X4: PLD-06, pds019_main_082_ext:PLD-06
- removed X6: (no value), pds019_main_082_ext:JP1
- added CON1: PINHEAD_2X03-PTH-2.54, pinhead:2X03-PTH-2.54
- added CON2: CON-5P-JST-VH, Connectors:B5P-VH
- added CON3, CON4: CON-2X3, degson:2EDGRHM-5.08-06P
- added IC1: TPS54231, dc-dc:SOIC8-POWERPAD
- added IC2: KPC357NT-SOP-4, misc:-SOP-4
- added LED1: LED-0805, rc:LED0805
- added X10: PINHEAD_1X02-2.54, pinhead:1X02-PTH-2.54
- BAT1: value CR2032 -> BATTERY-L-KLS5-CR2032-01; device pds019_main_082_ext:CR2032H-HOLD-1 -> mechanical:CR2032H
- C33, C34: device pds018:C1812 -> rc:C1812
- C89: device pds018:C0603 -> rc:C0603
- CN1: device pds019_main_082_ext:KF2EDGRM-7.62-03P -> degson:2EDGRM-7.62-03P
- CN10: device pds019:ST-033 -> Connectors:ST-033
- CN2: value B5P-VH -> CON-5P-JST-VH; device pds019_main_082_ext:JST_B5P_VH(-1) -> Connectors:B5P-VH
- CN4: value KF2EDGRHM-5.08-2X2P -> CON-2X2; device pds019_main_082_ext:KF2EDGRHM-5.08-2X2P -> degson:2EDGRHM-5.08-04P
- CN7, CN8: value COAX_FBNC_JR_CHN -> RF_CONNECTOR-BNC-KY-WE; device pds019:BNC_JR_CHN -> Connectors:BNC_JR_CHN
- D1, D5: device pds019:DO214AC -> TVS_diodes:DO-214AC(SMA)
- D6: device pds019_main_082_ext:DO214AC -> Diodes:DO-214AC(SMA)
- D8: device pds019_main_082_ext:SMB -> TVS_diodes:DO-214AA(SMB)
- F1, F2, F3, F4, F5, F6, F7, F8, F9: device pds019_main_082_ext:FC-001S -> rc:FC-001S
- F10: value 500mA -> FUSE-1206; device pds019_main_082_ext:F1206 -> rc:F1206
- F11: device pds019:F1206 -> rc:F1206
- K1, K2, K3, K4, K5: device pds019_main_082_ext:SRD_UNIV -> misc:SRD_UNIV
- Q4: device pds019:SOT23-GSD -> mosfet:SOT23
- U10: value 74LVC1G07 -> 74LVC1G07GV; device pds019:SOT23-5 -> misc:SOT23-5
- U11, U12, U15, U16: device pds019:SOT23-123 -> misc:SOT23B-3
- U13, U14: value AD8667R -> AD8667ARZ-SO8; device pds019:SO08 -> misc:SOIC8
- U17, U18: value MCP3551SN -> MCP3550; device pds019:SO08 -> misc:SOIC8
- U19, U20: value P2AU-0505ELF -> B0503S-1WR3; device pds018:SIP4_6X12 -> dc-dc:SIP-4
- U2: value ESP32-WROVER-E -> ESP32-WROVER-(I)E; device pds019_main_082_ext:ESP32-WROVER-E -> ali_modules:ESP32-WROVER-E
- U21, U22: device pds018:SO-16W -> serial_interfaces:SO-16W
- U25: device pds019_main_082_ext:SOT23-6 -> misc:SOT23-6
- U26: value 74AHCT1G125DBV -> SN74AHCT1G125DBVR-SOT23-5; device pds019_main_082_ext:SOT23-5 -> misc:SOT23-5
- U30, U8: device pds019:SOT23-5 -> misc:SOT23-5
- U31: device pds019:SOT23-6 -> misc:SOT23-6
- U7: device pds019:SO08 -> misc:SOIC8
- U9: device pds019_main_082_ext:SOT23-123 -> misc:SOT23B-3
- X1: value PLS-04 -> PINHEAD_1X04-2.54; device pds018:PLS-04 -> pinhead:1X04-PTH-2.54
- X2, X9: value (none) -> PINHEAD_1X02-2.54; device pds019_main_082_ext:JP1 -> pinhead:1X02-PTH-2.54
- X3: value PLS-05 -> PINHEAD_1X05-2.54; device pds019_main_082_ext:PLS-05 -> pinhead:1X05-PTH-2.54
- X5: value PLS-03 -> PINHEAD_1X03-2.54; device pds019:PLS-03 -> pinhead:1X03-PTH-2.54
- X7, X8: value PLS-03 -> PINHEAD_1X03-2.54; device pds019_main_082_ext:PLS-03 -> pinhead:1X03-PTH-2.54
- moved U2 8.25 mm to (-64.2, 71.2)
- moved U20 2.13 mm to (-73.0, -49.0)
- moved U19 2.08 mm to (-104.7, -49.0)
- turned D1 to 90 degrees
- turned D5 to 90 degrees
- turned D6 to 0 degrees
- turned D8 to 90 degrees
- turned Q4 to 90 degrees
- turned U10 to 90 degrees
- turned U21 to 270 degrees
- turned U22 to 270 degrees
- turned U25 to 90 degrees
- turned U26 to 270 degrees
- turned U30 to 270 degrees
- turned U31 to 90 degrees
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Connections:
- net +12V: now also IC1.2; no longer U4.2
- net +3V3: now also CON1.1, IC2.4, X1.4; no longer PC1.4, X1.1, X4.1
- net +5V: now also Q4.2; no longer Q4.S
- net AC_N: now also CON3.1.2, CON3.2.2, CON4.1.2, CON4.2.2; no longer CN5.1.2, CN5.2.2, CN6.1.2, CN6.2.2
- net ENC_BTN: now also X10.1; no longer X6.1
- net GND: now also CON1.6, IC1.7, IC1.POWERPAD, LED1.C, X1.1, X10.2; no longer HL17.K, U4.7, U4.EP, X1.4, X4.6, X6.2
- net LVL_24V: now also IC2.1; no longer PC1.1
- net N$10: now also LED1.A; no longer HL17.A
- net N$124: now also CON1.5; no longer X4.5
- net N$149: now also IC1.1; no longer U4.1
- net N$150: now also CON1.2; no longer X4.2
- net N$165: now also F11.P$2; no longer F11.2
- net N$19: now also X1.3; no longer X1.2
- net N$190: now also IC1.8; no longer U4.8
- net N$192: now also IC1.6; no longer U4.6
- net N$20: now also X1.2; no longer X1.3
- net N$204: now also CON4.1.1; no longer CN5.1.1
- net N$205: now also IC1.5; no longer U4.5
- net N$207: now also IC1.3; no longer U4.3
- net N$211: now also CON4.2.1; no longer CN5.2.1
- net N$213: now also CON1.3; no longer X4.3
- net N$214: now also CON3.1.1; no longer CN6.1.1
- net N$216: now also CON1.4; no longer X4.4
- net N$217: now also CON3.2.1; no longer CN6.2.1
- net N$23: now also IC2.2; no longer PC1.2
- net N$29: now also F11.P$1, Q4.3; no longer F11.1, Q4.D
- net N$49: no longer U2.28
- net N$50: no longer U2.27
- net N$64: now also F10.P$1; no longer F10.1
- net N$69: now also IC1.4; no longer U4.4
- net N$7: now also CON2.3; no longer CN3.3
- net N$77: now also Q4.1; no longer Q4.G
- net N$8: now also CON2.1; no longer CN3.1
- net N$89: no longer U8.1
- net N$96: now also F10.P$2; no longer F10.2
- net PE: now also CON2.5, CON3.1.3, CON3.2.3, CON4.1.3, CON4.2.3; no longer CN3.5, CN5.1.3, CN5.2.3, CN6.1.3, CN6.2.3
- net PE_PH: now also C33.P$2; no longer C33.2
- net PE_RX: now also C34.P$2; no longer C34.2
- net PH_VCOM: now also C33.P$1; no longer C33.1
- net RX_COM: now also C34.P$1; no longer C34.1
- net SENSOR_LEVEL: now also IC2.3; no longer PC1.3
Routing:
- net PE: track 565.1 -> 529.4 mm
- net N$49: track 4.95 -> 0.00 mm
- net KBD_13: track 86.6 -> 82.3 mm
- net N$50: track 3.18 -> 0.00 mm
- net N$69: track 5.04 -> 2.44 mm
- net RX_AMP_VO+: track 97.7 -> 95.5 mm
- net N$131: track 7.91 -> 5.77 mm
- net N$89: track 36.7 -> 34.9 mm
- net N$190: track 4.26 -> 3.18 mm
- net !NRST_205: track 23.8 -> 22.7 mm
- net PH_AMP_VO-: track 4.93 -> 5.97 mm
- net N$208: track 22.6 -> 23.6 mm
- net KBD_1: track 86.3 -> 85.3 mm
- net PH_VINF: track 5.68 -> 6.63 mm
- net GND: track 16.0 -> 15.1 mm
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
Commit message: its done now
Parts:
- removed CN9: USBA-KLS1-191-4P-0.7, pds019_main_082_ext:KLS1-191-4P-0.7
- removed K6: SLC-12VDC-SL-C, pds019_main_082_ext:SLC-12VDC-SL-C
- removed LCD1: LCD12864, pds019_main_082_ext:LCD12864_93X70_CHINA
- added CON5: USB-A-KLS1-191, Connectors:KLS1-191-4P-0.7
- added CON6: PINHEAD_1X20-2.54-MALE-LONG, pinhead:1X20-PTH-2.54-LONG
- added K7: SRD-SLC, misc:SLC-12VDC-SL-C
- added U$1: (no value), pds019:LCD12864_93X70_CHINA_SILK
- C108: value 4700pF 2kV -> 4700pF; device pds019_main_082_ext:C_5MM -> rc:C_5MM
- C35, C36: value 1000pF 2kV -> 1000pF; device pds019:C_5MM -> rc:C_5MM
- C59: value 100,0 25V -> 100,0; device pds019_main_082_ext:CTANT_7X4 -> rc:CTANT_7X4
- C60: value 100,0 6V3 -> 100,0; device pds019_main_082_ext:CTANT_B -> rc:CTANT_B
- C72: value 150,0 16V -> 150,0; device pds019_main_082_ext:CTANT_7X4 -> rc:CTANT_7X4
- C90: value 4700pF 2kV -> 4700pF; device pds019:C_5MM -> rc:C_5MM
- CN12: device pds019_main_082_ext:IDC_2X05 -> Connectors:IDC_2X05
- CN13: device pds019_main_082_ext:IDC_2X07 -> Connectors:IDC_2X07
- ENC1: device pds019_main_082_ext:PEC12R-4XXXF-SXXXX -> misc:PEC12R-4XXXF-SXXXX
- L1: value 22uH 0630 -> 22uH; device pds019_main_082_ext:LSMD_06030 -> power_inductors:LSMD_06030
- L2: value 2,2uH 0520 -> 3.3uH; device pds019_main_082_ext:LSMD_05020 -> power_inductors:LSMD_05020
- Q1, Q2, Q3: device pds018:SOT23-BEC -> misc:SOT23B-3
- SB1: device pds019_main_082_ext:SW4-6.0X6.0X5.0MM -> mechanical:SW4-6.0X6.0X5.0MM
- U1: device pds019_main_082_ext:LQFP64_0.5_10X10_STM_MIL -> stm32:TQFP64
- U6: device pds019:SIP7_6X19.65_SINGLE -> dc-dc:SIP7_6X19.65_SINGLE
- VR1: device pds019_main_082_ext:S20K420 -> rc:S20K420
- Z1: value 25MHz 3225 -> 25MHz; device pds019_main_082_ext:XTAL_3225_4PIN -> crystal:OSCILLATOR-3.2X2.5-4P
- Z2: value 32K 3215 -> 32K; device pds019_main_082_ext:XTAL_3215 -> crystal:32X15
- moved TP18 0.18 mm to (-58.8, -30.7)
- turned U1 to 270 degrees
Connections:
- net !LCD_RST: now also CON6.17; no longer LCD1.17
- net +12V: now also K7.C2; no longer K6.C2
- net AC_L: now also K7.COM; no longer K6.COM
- net BUZZER_PWM: now also Q1.1, Q3.1; no longer Q1.B, Q3.B
- net GND: now also CON5.4, CON5.SH1, CON5.SH2, CON5.SH3, CON5.SH4, CON6.1, CON6.15, Q1.2, Q2.2, Q3.2; no longer CN9.4, CN9.SH1, CN9.SH2, CN9.SH3, CN9.SH4, LCD1.1, LCD1.15, Q1.E, Q2.E, Q3.E
- net LCD_CS: now also CON6.4; no longer LCD1.4
- net LCD_DATA: now also CON6.5; no longer LCD1.5
- net LCD_LED: now also Q2.1; no longer Q2.B
- net LCD_LED_A: now also CON6.19; no longer LCD1.19
- net LCD_LED_K: now also CON6.20, Q2.3; no longer LCD1.20, Q2.C
- net LCD_V0: now also CON6.3; no longer LCD1.3
- net LCD_VEE: now also CON6.18; no longer LCD1.18
- net N$125: now also CON5.2; no longer CN9.2
- net N$131: now also CON5.3; no longer CN9.3
- net N$18: now also CON6.6; no longer LCD1.6
- net N$183: now also K7.NO; no longer K6.NO
- net N$197: now also Q1.3; no longer Q1.C
- net N$30: now also CON6.2; no longer LCD1.2
- net N$39: now also K7.C1; no longer K6.C1
- net N$64: now also CON5.1; no longer CN9.1
- net N$75: now also Q3.3; no longer Q3.C
- net RTC_XTAL_IN: now also Z2.P$2; no longer Z2.2
- net RTC_XTAL_OUT: now also Z2.P$1; no longer Z2.1
Routing:
- net +5V: track 1067.1 -> 1050.2 mm
- net BUZZER_PWM: track 187.1 -> 174.6 mm
- net +12V: track 351.3 -> 341.1 mm
- net N$39: track 169.1 -> 161.7 mm
- net N$116: track 71.6 -> 64.6 mm
- net N$175: track 136.5 -> 130.0 mm
- net N$164: track 117.5 -> 111.5 mm
- net N$170: track 98.5 -> 92.8 mm
- net +3V3: track 698.6 -> 693.0 mm
- net N$8: track 109.0 -> 103.4 mm
- net PE: track 529.4 -> 524.1 mm
- net N$112: track 79.5 -> 74.7 mm
- net N$214: track 43.7 -> 39.1 mm
- net ESP32_STM_SWCLK: track 107.3 -> 103.4 mm
- net ESP32_RXD0: track 121.5 -> 118.0 mm
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Other:
- board text added: "23/03/2026"
- board text added: "PDS019_MAIN_PRETTY"
- board text added: "REV: 0.92"
- board text removed: "03/07/2023"
- board text removed: "PDS019_MAIN"
- board text removed: "REV: 0.82"

Commit message: Update pds019_main_082_ext.brd
Parts:
- added U$2: (no value), pds019:ART
